File: HARDWARE/MAIN-BOARD/KOSMO-POLY6-PICO-DCO-MB.kicad_pcb (KiCad board)
At the start: 2 copper layers, 95 x 175 mm, 167 parts, among them Q1 2N3904, Q2 2N3904, Q3 2N3904, Q4 2N3904, Q5 2N3904, Q6 2N3904, Q7 2N3904, U1 L7805, U2 TL074, U3 H11L1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

Commit message: baord ready
Parts:
- moved MCU1 5.83 mm to (92.6, 138.9)
Routing:
- net GND: track 857.4 -> 0.00 mm
- net +12V: track 410.7 -> 0.00 mm
- net -12V: track 388.9 -> 0.00 mm
- net Net-(H1-Pad1): track 342.3 -> 0.00 mm
- net PW_POT: track 261.9 -> 0.00 mm
- net PWM_IN: track 257.3 -> 0.00 mm
- net +3V3: track 197.2 -> 0.00 mm
- net +5V: track 188.4 -> 0.00 mm
- net RANGE_PWM0: track 139.5 -> 0.00 mm
- net RAMP_OUT4: track 125.7 -> 0.00 mm
- net RESET1: track 113.9 -> 0.00 mm, vias 1 -> 0
- net RANGE_PWM1: track 111.7 -> 0.00 mm
- net GATE_OUT0: track 108.1 -> 0.00 mm, vias 1 -> 0
- net GATE_OUT1: track 104.2 -> 0.00 mm
- net PULSE_OUT4: track 101.9 -> 0.00 mm
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Other:
- net class Audio Path added: clearance 0.8, trace_width 0.25, via_dia 0.8, via_drill 0.4

Commit message: sync
Parts:
- added C36: 100n, Capacitor_THT:C_Rect_L7.2mm_W4.5mm_P5.00mm_FKS2_FKP2_MKS2_MKP2, F.Cu at (123.6, 48.6)
- added C37: 100n, Capacitor_THT:C_Rect_L7.2mm_W4.5mm_P5.00mm_FKS2_FKP2_MKS2_MKP2, F.Cu at (83.7, 48.9)
- added C38: 100n, Capacitor_THT:C_Rect_L7.2mm_W4.5mm_P5.00mm_FKS2_FKP2_MKS2_MKP2, F.Cu at (123.1, 79.9)
- added C39: 100n, Capacitor_THT:C_Rect_L7.2mm_W4.5mm_P5.00mm_FKS2_FKP2_MKS2_MKP2, F.Cu at (83.7, 79.9)
- added C40: 100n, Capacitor_THT:C_Rect_L7.2mm_W4.5mm_P5.00mm_FKS2_FKP2_MKS2_MKP2, F.Cu at (123.5, 111.4)
- added C41: 100n, Capacitor_THT:C_Rect_L7.2mm_W4.5mm_P5.00mm_FKS2_FKP2_MKS2_MKP2, F.Cu at (84.0, 112.0)
- moved R36 15.7 mm to (134.0, 84.0), turned to 270 degrees
- moved C30 15.5 mm to (114.7, 111.4), turned to 0 degrees
- moved R6 15.4 mm to (133.8, 52.3), turned to 270 degrees
- moved C15 15.1 mm to (75.1, 48.8), turned to 0 degrees
- moved C20 14.9 mm to (115.2, 79.9), turned to 0 degrees
- moved C35 14.6 mm to (75.9, 112.1), turned to 0 degrees
- moved C25 14.6 mm to (75.8, 80.1), turned to 0 degrees
- moved C5 14.4 mm to (115.7, 48.6), turned to 0 degrees
- moved R50 10.5 mm to (87.3, 86.4)
- moved R22 10.5 mm to (86.9, 55.3)
- moved R78 10.2 mm to (87.6, 117.6)
- moved R64 9.38 mm to (125.9, 117.5)
- moved R62 7.65 mm to (133.8, 116.2), turned to 90 degrees
- moved R34 7.01 mm to (129.0, 86.6)
- moved R3 6.45 mm to (127.8, 54.8)
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Connections:
- net RX renamed Net-(MCU1-Pad2)
- C15 pad 1: +12V -> GND
- C15 pad 2: -12V -> +12V
- C20 pad 1: +12V -> GND
- C20 pad 2: -12V -> +12V
- C25 pad 1: +12V -> GND
- C25 pad 2: -12V -> +12V
- C30 pad 1: +12V -> GND
- C30 pad 2: -12V -> +12V
- C35 pad 1: +12V -> GND
- C35 pad 2: -12V -> +12V
- C5 pad 1: +12V -> GND
- C5 pad 2: -12V -> +12V
Routing:
- net GND: track 0.00 -> 903.2 mm
- net -12V: track 0.00 -> 400.4 mm
- net +12V: track 0.00 -> 381.9 mm
- net Net-(H1-Pad1): track 0.00 -> 343.6 mm
- net PW_POT: track 0.00 -> 266.0 mm
- net PWM_IN: track 0.00 -> 264.4 mm
- net RANGE_PWM0: track 0.00 -> 240.4 mm
- net +5V: track 0.00 -> 184.1 mm
- net +3V3: track 0.00 -> 182.5 mm
- net RAMP_OUT4: track 0.00 -> 146.9 mm, vias 0 -> 1
- net RANGE_PWM1: track 0.00 -> 141.9 mm, vias 0 -> 2
- net RAMP_OUT2: track 0.00 -> 141.5 mm
- net PULSE_OUT2: track 0.00 -> 137.3 mm, vias 0 -> 1
- net GATE_OUT3: track 0.00 -> 129.7 mm
- net RAMP_OUT5: track 0.00 -> 127.6 mm
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Other:
- board text added: "KOSMO-POLY6-PICO-DCO - By TwinTurbo V0.1.1 Credit Original Design Polykit"
- board text removed: "Mainboard KosmoDCO - By TwinTurbo V0.1.0 Credit Original Design Polykit"

Commit message: Added jumper on PWM pot to go to future PG Programmer
Parts:
- added PG1: TO PG, Jumper if not used, Connector_Molex:Molex_KK-254_AE-6410-02A_1x02_P2.54mm_Vertical, F.Cu at (92.5, 176.1)
Connections:
- PW_POT1 pad 2: PW_POT -> Net-(PG1-Pad2)
Routing:
- net PW_POT: track 266.0 -> 275.7 mm
- net Net-(PG1-Pad2): track 0.00 -> 8.55 mm
